File: prophet.kicad_pcb (KiCad board)
At the start: 2 copper layers, 285.8 x 94.5 mm, 113 parts, among them U1 STM32F072CBTx

Commit message: added new updates
Routing:
- net (no net): track 0.00 -> 312.5 mm, vias 0 -> 2
Changed lines of the file:
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@@
     (thickness 1.6)
     (drawings 40)
-    (tracks 1160)
+    (tracks 1180)
     (zones 0)
     (modules 153)
@@
   (gr_line (start 73.025 95.25) (end 73.025 184.94375) (layer Edge.Cuts) (width 0.15))
   (gr_line (start 356.39375 92.86875) (end 75.40625 92.86875) (layer Edge.Cuts) (width 0.15))
+  (segment (start 171.179542 174.418629) (end 171.116629 174.418629) (width 0.254) (layer B.Cu) (net 0))
+  (via (at 167.4368 173.6344) (size 0.6) (drill 0.4) (layers F.Cu B.Cu) (net 0))
+  (segment (start 171.116629 174.418629) (end 170.3324 173.6344) (width 0.254) (layer B.Cu) (net 0))
+  (segment (start 170.3324 173.6344) (end 167.4368 173.6344) (width 0.254) (layer B.Cu) (net 0))
+  (segment (start 171.533095 174.065076) (end 171.525076 174.065076) (width 0.254) (layer B.Cu) (net 0))
+  (via (at 167.9448 172.72) (size 0.6) (drill 0.4) (layers F.Cu B.Cu) (net 0))
+  (segment (start 171.525076 174.065076) (end 170.18 172.72) (width 0.254) (layer B.Cu) (net 0))
+  (segment (start 170.18 172.72) (end 167.9448 172.72) (width 0.254) (layer B.Cu) (net 0))
+  (segment (start 76.6572 111.9632) (end 80.8228 107.7976) (width 0.254) (layer F.Cu) (net 0))
+  (segment (start 76.6572 179.07) (end 76.6572 111.9632) (width 0.254) (layer F.Cu) (net 0))
+  (segment (start 83.4136 185.8264) (end 76.6572 179.07) (width 0.254) (layer F.Cu) (net 0))
+  (segment (start 150.6728 185.8264) (end 83.4136 185.8264) (width 0.254) (layer F.Cu) (net 0))
+  (segment (start 167.4368 173.6344) (end 162.8648 173.6344) (width 0.254) (layer F.Cu) (net 0))
+  (segment (start 162.8648 173.6344) (end 150.6728 185.8264) (width 0.254) (layer F.Cu) (net 0))
+  (segment (start 77.1652 152.3492) (end 82.4484 147.066) (width 0.254) (layer F.Cu) (net 0))
+  (segment (start 77.1652 178.8668) (end 77.1652 152.3492) (width 0.254) (layer F.Cu) (net 0))
+  (segment (start 83.6168 185.3184) (end 77.1652 178.8668) (width 0.254) (layer F.Cu) (net 0))
+  (segment (start 150.5204 185.3184) (end 83.6168 185.3184) (width 0.254) (layer F.Cu) (net 0))
+  (segment (start 167.9448 172.72) (end 163.1188 172.72) (width 0.254) (layer F.Cu) (net 0))
+  (segment (start 163.1188 172.72) (end 150.5204 185.3184) (width 0.254) (layer F.Cu) (net 0))
   (segment (start 87.755 97.62531) (end 88.81219 98.6825) (width 0.635) (layer B.Cu) (net 1))
   (segment (start 87.755 97.2675) (end 87.755 97.62531) (width 0.635) (layer B.Cu) (net 1))
