File: prophet.sch (KiCad schematic (older format))
At the start: 19 parts, among them Q1 Q_NPN_BCE, SW1 , U1 STM32F072CBTx, U2 LD3985G33R_TSOT23, U3 PRTR5V0U2X

Commit message: update to latest rev
Parts:
- removed U3: PRTR5V0U2X, Package_TO_SOT_SMD:SOT143B, symbol ai03-locallib:PRTR5V0U2X
- added U3: PRTR5V0U2X, random-keyboard-parts:SOT143B, symbol random-keyboard-parts:PRTR5V0U2X
- C3, C4, C5, C6, C7, C8, C9: footprint Capacitor_SMD:C_0805_2012Metric_Pad1.15x1.40mm_HandSolder -> Diode_SMD:D_0805_2012Metric
- DR1: footprint Diode_SMD:D_0805_2012Metric_Pad1.15x1.40mm_HandSolder -> Diode_SMD:D_0805_2012Metric
- F1: footprint Fuse:Fuse_0805_2012Metric_Pad1.15x1.40mm_HandSolder -> Fuse:Fuse_0805_2012Metric
- Q1: value Q_NPN_BCE -> BC850; footprint TO_SOT_Packages_SMD:SOT-23 -> Package_TO_SOT_SMD:SOT-23
- R1, R2, R6, R7: footprint Resistor_SMD:R_0805_2012Metric_Pad1.15x1.40mm_HandSolder -> Resistor_SMD:R_0805_2012Metric
- SW1: footprint Button_Switch_SMD:SKSVCAE010 -> reset:ResetShort
Connections:
- net GND: now also U3.1 (GND)
- net USB+: now also U3.2 (IO1)
- net USB-: now also U3.3 (IO2)
- net VCC: now also U3.4 (VCC)
- net ESC_LED: now reaches U1.25 (PB12)
- net CAPS_LED: now reaches U1.26 (PB13)
- no-connect marks 18 -> 16
Other:
- moved on the sheet: U1
