File: ccd60.sch (KiCad schematic (older format))
At the start: 20 parts, among them Q1 BC850, SW1 , U1 STM32F072CBTx, U2 LD3985G33R_TSOT23, U3 PRTR5V0U2X

Commit message: updated to latest rev
Parts:
- added H2, H3, H4, H5, H6, H7: ScrewHole, cablecardesigns:m2-oval, symbol Mechanical:MountingHole_Pad
- added JST1: JST-SH Header, Connector_JST:JST_SH_SM04B-SRSS-TB_1x04-1MP_P1.00mm_Horizontal, symbol Connector_Generic_MountingPin:Conn_01x04_MountingPin
Connections:
- net GND: now also H2.1, H3.1, H4.1, H5.1, H6.1, H7.1, JST1.4 (Pin_4), JST1.MP (MountPin)
- net USB+: now also JST1.3 (Pin_3)
- net USB-: now also JST1.2 (Pin_2)
- net VCC: now also JST1.1 (Pin_1)
Other:
- note added: "JST Header\n"
- note added: "Mounting Holes\n"
- moved on the sheet: U1
