File: ccd60_matrix.sch (KiCad schematic (older format))
At the start: 134 parts

Commit message: updated to latest rev
Parts:
- renumbered D58 to D10, D3 to D11, D17 to D12, D31 to D13, D45 to D14, D59 to D15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
Connections:
- net CAPS_LED: now also MX_2.4 (LEDGND), MX_29_1.4 (LEDGND); no longer RMX1.2
- net ESC_LED: now also MX_1.4 (LEDGND); no longer RMX2.1
- removed net GND: MX_1.4 (LEDGND), MX_2.4 (LEDGND), MX_29_1.4 (LEDGND)
- new net +5V: RMX1.2, RMX2.1
